Commit message: Searchin with dynamic overestimation

File: rotors_description/urdf/depth_camera_base.xacro (robot description, xacro)
@@ -42,5 +42,5 @@
         <mass value="0" />
         <origin xyz="0 0 0" rpy="0 0 0"/>
-        <inertia ixx="1e-6" ixy="0" ixz="0" iyy="1e-6" iyz="0" izz="1e-6" />
+        <inertia ixx="1e-7" ixy="0" ixz="0" iyy="1e-7" iyz="0" izz="1e-7" />
       </inertial>
     </link>

Commit message: Collision detection and goBack fix

File: rotors_description/urdf/depth_camera_base.xacro (robot description, xacro)
@@ -42,5 +42,5 @@
         <mass value="0" />
         <origin xyz="0 0 0" rpy="0 0 0"/>
-        <inertia ixx="1e-7" ixy="0" ixz="0" iyy="1e-7" iyz="0" izz="1e-7" />
+        <inertia ixx="1e-8" ixy="0" ixz="0" iyy="1e-8" iyz="0" izz="1e-8" />
       </inertial>
     </link>
